File: Chorus_Caeruleus.kicad_sch (KiCad schematic)
At the start: 125 parts, among them Q1 2N5088, Q10 J201, Q11 J201, Q2 2N5088, Q3 2N5088, Q4 2N5088, Q5 2N5088, Q7 2SC1815, Q8 2SC1815, Q9 2SC1815, SW1 SW_Push, SW2 SW_SPST, U1 RC4558, U2 MN3207, U3 MN3102, U4 TL022

Commit message: Proj renamed, PCB upd
Parts:
- renumbered C15 to C44, C44 to C45, C62 to C61, C61 to C62, Q5 to Q2, Q2 to Q5, Q9 to Q6, Q11 to Q9, R65 to R64, R64 to R65
Changed lines of the file:
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@@
 		(in_pos_files yes)
 		(dnp no)
-		(property "Reference" "R65"
+		(property "Reference" "R64"
 			(at 233.045 119.38 0)
 			(show_name no)
@@
 			(project "Azure_chorus"
 				(path "/738e02f3-8b44-4a7f-854b-b4c60cc26898"
-					(reference "R65")
+					(reference "R64")
 					(unit 1)
 				)
@@
 		(in_pos_files yes)
 		(dnp no)
-		(property "Reference" "R64"
+		(property "Reference" "R65"
 			(at 254.635 119.38 0)
 			(show_name no)
@@
 			(project "Azure_chorus"
 				(path "/738e02f3-8b44-4a7f-854b-b4c60cc26898"
-					(reference "R64")
+					(reference "R65")
 					(unit 1)
 				)
@@
 		(in_pos_files yes)
 		(dnp no)
-		(property "Reference" "C44"
+		(property "Reference" "C45"
 			(at 125.73 103.505 90)
 			(show_name no)
@@
 			(project "Azure_chorus"
 				(path "/738e02f3-8b44-4a7f-854b-b4c60cc26898"
-					(reference "C44")
+					(reference "C45")
 					(unit 1)
 				)
@@
 		(in_pos_files yes)
 		(dnp no)
-		(property "Reference" "Q5"
+		(property "Reference" "Q2"
 			(at 165.735 139.7001 0)
 			(show_name no)
@@
 			(project "Azure_chorus"
 				(path "/738e02f3-8b44-4a7f-854b-b4c60cc26898"
-					(reference "Q5")
+					(reference "Q2")
 					(unit 1)
 				)
@@
 		(in_pos_files yes)
 		(dnp no)
-		(property "Reference" "Q9"
+		(property "Reference" "Q6"
 			(at 210.312 106.426 0)
 			(show_name no)
@@
 			(project "Azure_chorus"
 				(path "/738e02f3-8b44-4a7f-854b-b4c60cc26898"
-					(reference "Q9")
+					(reference "Q6")
 					(unit 1)
 				)
@@
 		(in_pos_files yes)
 		(dnp no)
-		(property "Reference" "C61"
-			(at 239.649 119.888 0)
+		(property "Reference" "C62"
+			(at 239.395 119.38 0)
 			(show_name no)
 			(do_not_autoplace no)
@@
 			(project "Azure_chorus"
 				(path "/738e02f3-8b44-4a7f-854b-b4c60cc26898"
-					(reference "C61")
+					(reference "C62")
 					(unit 1)
 				)
@@
 		(in_pos_files yes)
 		(dnp no)
-		(property "Reference" "C15"
+		(property "Reference" "C44"
 			(at 144.272 86.36 0)
 			(show_name no)
@@
 			(project "Azure_chorus"
 				(path "/738e02f3-8b44-4a7f-854b-b4c60cc26898"
-					(reference "C15")
+					(reference "C44")
 					(unit 1)
 				)
@@
 		(in_pos_files yes)
 		(dnp no)
-		(property "Reference" "Q11"
+		(property "Reference" "Q9"
 			(at 233.045 67.564 90)
 			(show_name no)
@@
 			(project "Azure_chorus"
 				(path "/738e02f3-8b44-4a7f-854b-b4c60cc26898"
-					(reference "Q11")
+					(reference "Q9")
 					(unit 1)
 				)
@@
 		(in_pos_files yes)
 		(dnp no)
-		(property "Reference" "Q2"
+		(property "Reference" "Q5"
 			(at 73.66 127.254 0)
 			(show_name no)
@@
 			(project "Azure_chorus"
 				(path "/738e02f3-8b44-4a7f-854b-b4c60cc26898"
-					(reference "Q2")
+					(reference "Q5")
 					(unit 1)
 				)
@@
 		(in_pos_files yes)
 		(dnp no)
-		(property "Reference" "C62"
-			(at 248.031 119.888 0)
+		(property "Reference" "C61"
+			(at 248.285 119.38 0)
 			(show_name no)
 			(do_not_autoplace no)
@@
 			(project "Azure_chorus"
 				(path "/738e02f3-8b44-4a7f-854b-b4c60cc26898"
-					(reference "C62")
+					(reference "C61")
 					(unit 1)
 				)

Commit message: PCB upd
Connections:
- net VC: now also DEPTH1.3, R71.2; no longer DEPTH1.1, R71.1
- net at C58.2, R54.2, U4.7: now also DEPTH1.1; no longer DEPTH1.3
- net at C70.2, Q9.1 (D): now also R71.1; no longer R71.2
- net at R55.2, U4.1: now also RATE1.1; no longer RATE1.3
- net at R56.1: now also RATE1.3; no longer RATE1.1
Other:
- moved on the sheet: C10, C11, C12, C20, C21, C22, C30, C31, C32, C33, C40, C41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

Commit message: PCB upd
Parts:
- D5: footprint LED_THT:LED_D3.0mm -> Connector_PinHeader_2.00mm:PinHeader_1x02_P2.00mm_Vertical
Changed lines of the file:
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@@
 			)
 		)
-		(property "Footprint" "LED_THT:LED_D3.0mm"
+		(property "Footprint" "Connector_PinHeader_2.00mm:PinHeader_1x02_P2.00mm_Vertical"
 			(at 193.04 118.11 0)
 			(hide yes)
