File: Chorus_Caeruleus.kicad_pcb (KiCad board)
At the start: 2 copper layers, 55 x 80 mm, 125 parts, among them Q1 2N5088, Q10 J201, Q11 J201, Q2 2N5088, Q3 2N5088, Q4 2N5088, Q5 2N5088, Q7 2SC1815, Q8 2SC1815, Q9 2SC1815, SW1 SW_Push, SW2 SW_SPST, U1 RC4558, U2 MN3207, U3 MN3102, U4 TL022

Commit message: Proj renamed, PCB upd
Parts:
- moved C20 126.6 mm to (60.6, 90.7), turned to 90 degrees
- moved C21 124.5 mm to (63.6, 91.6)
- moved C22 124.5 mm to (63.6, 95.0)
- moved C11 119.6 mm to (87.0, 81.0), turned to 180 degrees
- moved CE1 107.2 mm to (108.2, 76.5), turned to -90 degrees
- moved CE3 106.9 mm to (108.2, 82.9), turned to 90 degrees
- moved C12 106.1 mm to (82.0, 84.0)
- moved Q1 104.3 mm to (89.5, 77.9), turned to 90 degrees
- moved R1 100.6 mm to (239.7, 71.5)
- moved Q6 99.7 mm to (100.1, 79.6), turned to -90 degrees
- moved R69 99.4 mm to (263.1, 132.9)
- moved R67 99.4 mm to (263.1, 124.8)
- moved R25 98.3 mm to (52.2, 94.8)
- moved R26 98.3 mm to (52.2, 98.8)
- moved C50 96.0 mm to (214.7, 31.8)
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- renumbered C15 to C44, C44 to C45, C62 to C61, C61 to C62, Q5 to Q2, Q2 to Q5, Q9 to Q6, Q11 to Q9, R65 to R64, R64 to R65
Routing:
- net /VC: track 0.00 -> 73.9 mm, vias 0 -> 1
- net /VA: track 0.00 -> 45.5 mm, vias 0 -> 1
- net Net-(U2-VGG): track 0.00 -> 26.8 mm
- net Net-(Q10-S): track 0.00 -> 20.3 mm
- net Net-(Q10-D): track 0.00 -> 18.8 mm
- net /RC_OUT: track 0.00 -> 16.7 mm
- net /VD: track 0.00 -> 16.2 mm
- net Net-(SW2-B): track 0.00 -> 15.9 mm
- net /IN: track 0.00 -> 11.7 mm
- net /Q4_1: track 0.00 -> 11.6 mm
- net Net-(U2-CP1): track 0.00 -> 10.7 mm
- net Net-(Q10-G): track 0.00 -> 9.97 mm
- net Net-(D1-K): track 0.00 -> 8.05 mm
- net Net-(Q6-C): track 0.00 -> 7.73 mm
- net Net-(R57-Pad1): track 0.00 -> 7.36 mm
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Other:
- board size 55 x 80 mm -> 54 x 80 mm
- board text added: "DC1"
- board text added: "DEPTH1"
- board text added: "IN1"
- board text added: "MIX1"
- board text added: "OUT1"
- board text added: "RATE1"
- board text added: "SW2"

Commit message: PCB upd
Parts:
- moved CE2 166.9 mm to (91.3, 158.3)
- moved R1 166.7 mm to (91.5, 147.9)
- moved Z1 166.7 mm to (92.5, 152.9)
- moved Q8 156.2 mm to (122.0, 135.2)
- moved C61 155.2 mm to (113.2, 124.7), turned to 90 degrees
- moved Q7 153.2 mm to (124.5, 124.8), turned to 180 degrees
- moved C60 152.4 mm to (110.4, 135.7), turned to -90 degrees
- moved C62 149.3 mm to (113.2, 135.7), turned to -90 degrees
- moved R60 147.6 mm to (103.1, 132.3), turned to 180 degrees
- moved R61 147.4 mm to (103.1, 135.3), turned to 180 degrees
- moved R62 147.2 mm to (103.1, 138.3), turned to 180 degrees
- moved R67 144.9 mm to (118.9, 138.7), turned to 90 degrees
- moved C63 144.0 mm to (124.5, 128.8), turned to 180 degrees
- moved C64 143.9 mm to (124.5, 131.2), turned to 180 degrees
- moved R63 141.1 mm to (107.7, 128.1), turned to -90 degrees
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Connections:
- DEPTH1 pad 1: /VC -> Net-(C58-Pad2)
- DEPTH1 pad 3: Net-(C58-Pad2) -> /VC
- R71 pad 1: /VC -> Net-(Q9-D)
- R71 pad 2: Net-(Q9-D) -> /VC
- RATE1 pad 1: Net-(R56-Pad1) -> Net-(R55-Pad2)
- RATE1 pad 3: Net-(R55-Pad2) -> Net-(R56-Pad1)
Routing:
- net Net-(R55-Pad2): track 0.00 -> 52.0 mm, vias 0 -> 2
- net Net-(Q6-C): track 7.73 -> 57.8 mm
- net /OFF: track 0.00 -> 47.5 mm, vias 0 -> 1
- net /ON: track 0.00 -> 46.8 mm
- net Net-(Q5-B): track 0.00 -> 43.2 mm, vias 0 -> 2
- net Net-(U4B--): track 0.00 -> 39.6 mm, vias 0 -> 2
- net Net-(C58-Pad2): track 0.00 -> 39.4 mm, vias 0 -> 1
- net /U1_6: track 3.35 -> 41.5 mm
- net /PR_IN: track 6.60 -> 40.4 mm
- net /RC_OUT: track 16.7 -> 47.5 mm
- net Net-(D6-A): track 0.00 -> 26.3 mm
- net Net-(C60-Pad1): track 0.00 -> 18.7 mm
- net Net-(Q8-B): track 0.00 -> 17.0 mm
- net /VA: track 45.5 -> 62.3 mm
- net /LFO: track 4.63 -> 19.8 mm
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
Commit message: PCB upd
PCB routed
Parts:
- moved R5 49.7 mm to (80.7, 125.9), turned to 90 degrees
- moved R44 49.5 mm to (121.0, 107.3), turned to -90 degrees
- moved C41 47.5 mm to (115.3, 114.9), turned to 90 degrees
- moved C42 47.1 mm to (123.7, 108.9), turned to 0 degrees
- moved R43 44.4 mm to (118.0, 114.8), turned to 90 degrees
- moved CE4 44.0 mm to (116.9, 118.0)
- moved 3296W1 43.2 mm to (98.4, 127.2), turned to 180 degrees
- moved CE2 37.6 mm to (85.6, 121.1), turned to -90 degrees
- moved C43 34.6 mm to (128.9, 108.9), turned to 0 degrees
- moved R45 32.3 mm to (131.2, 111.6), turned to 180 degrees
- moved C44 31.4 mm to (131.7, 97.3), turned to -90 degrees
- moved C45 29.4 mm to (124.5, 97.3), turned to -90 degrees
- moved R47 28.9 mm to (131.9, 106.2), turned to 180 degrees
- moved Q4 28.7 mm to (128.4, 100.2), turned to 90 degrees
- moved R48 28.4 mm to (124.5, 94.7), turned to 0 degrees
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Routing:
- net /VA: track 62.3 -> 181.8 mm, vias 1 -> 2
- net /VB: track 0.00 -> 117.9 mm, vias 0 -> 1
- net /VC: track 72.9 -> 153.3 mm, vias 1 -> 2
- net /VD: track 16.2 -> 57.4 mm
- net /RC_IN: track 3.97 -> 44.9 mm
- net /U2_OUT: track 5.59 -> 26.8 mm
- net Net-(3296W1-Pad1): track 0.00 -> 17.8 mm
- net /ON: track 46.8 -> 55.8 mm
- net Net-(3296W1-Pad3): track 0.00 -> 7.69 mm
- net /MN_IN: track 0.00 -> 6.82 mm
- net Net-(C43-Pad1): track 4.92 -> 11.6 mm
- net Net-(C32-Pad1): track 0.00 -> 5.74 mm
- net /Q5_1: track 3.00 -> 6.81 mm
- net Net-(R57-Pad1): track 4.31 -> 7.82 mm
- net Net-(Q2-B): track 0.00 -> 3.44 mm
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
Commit message: PCB upd
Parts:
- D5: footprint LED_THT:LED_D3.0mm -> Connector_PinHeader_2.00mm:PinHeader_1x02_P2.00mm_Vertical
- moved D5 0.32 mm to (99.2, 61.8), turned to 90 degrees
- moved R46 0.30 mm to (131.9, 103.2)
- moved R13 0.11 mm to (97.0, 80.5)
- moved R3 0.10 mm to (104.5, 75.9)
- moved C11 0.10 mm to (87.0, 80.5)
- moved C12 0.10 mm to (82.0, 83.6)

Commit message: PCB upd
added teardrops
Parts:
- moved R53 3.20 mm to (99.4, 66.1)
- moved R0 3.00 mm to (96.2, 73.7)
- moved D5 0.84 mm to (100.0, 61.5)
- moved R5 0.59 mm to (80.7, 126.5)
- moved R70 0.55 mm to (117.8, 94.7)
- moved C70 0.55 mm to (117.8, 84.8)
- moved C71 0.33 mm to (121.0, 99.7)
- moved R71 0.33 mm to (120.8, 80.0)
- moved R72 0.33 mm to (120.8, 89.8)
- moved R12 0.31 mm to (93.1, 76.3)
- moved R23 0.20 mm to (102.4, 66.1)
- moved R24 0.20 mm to (105.8, 73.7)
- moved R14 0.19 mm to (98.2, 83.5)
- moved R22 0.19 mm to (101.2, 83.5)
- moved R44 0.19 mm to (121.0, 107.5)
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Routing:
- net /VC: track 153.5 -> 159.3 mm
- net Net-(DEPTH1-Pad2): track 5.38 -> 8.01 mm
- net /U2_OUT: track 26.8 -> 29.3 mm
- net Net-(Q5-B): track 42.6 -> 40.4 mm, vias 2 -> 1
- net /OFF: track 48.4 -> 46.5 mm
- net Net-(D5-K): track 4.35 -> 6.17 mm
- net Net-(Q6-C): track 61.0 -> 62.4 mm
- net /VD: track 57.2 -> 58.0 mm
- net Net-(D6-A): track 26.3 -> 26.8 mm
- net /VA: track 182.2 -> 182.7 mm
- net GND: vias 0 -> 1
